File: slave.brd (EAGLE design)
At the start: 217 x 21 mm, 11 parts, among them IC1 74HC574N

Commit message: final version prototype
Parts:
- C1: value (none) -> 0.1u
Connections:
- net VCC: now also SV1.4
Routing:
- net N$8: track 197.9 -> 202.7 mm, vias 1 -> 0
- net VCC: track 45.8 -> 49.4 mm
- net N$2: track 37.4 -> 40.9 mm, vias 1 -> 0
- net N$7: track 171.2 -> 171.5 mm, vias 1 -> 0
- net N$6: track 144.4 -> 144.6 mm, vias 1 -> 0
- net N$5: track 117.6 -> 117.8 mm, vias 1 -> 0
- net N$1: track 11.6 -> 11.5 mm, vias 1 -> 0
- net N$4: vias 1 -> 0
- net N$3: vias 1 -> 0
- removed copper zone on layer 1, net IC
- removed copper zone on layer 16, net J
- removed copper zone on layer 16, net P
Other:
- board text added: "4"
- board text added: "CLK"
